File: BerkerOgPower.kicad_pcb (KiCad board)
At the start: 2 copper layers, 99.2 x 98.6 mm, 63 parts, among them J1 +3,31V, J10 D4, J11 Screw_Terminal_01x03, J12 A0, J13 Conn_01x02, J14 Conn_01x03, J2 +5.1V, J3 GND, J4 D4, J5 Screw_Terminal_01x03, J6 A0, J7 +3,32V, J8 +5.2V, J9 GND, K1 SANYOU_SRD_Form_C, K2 SANYOU_SRD_Form_C, M3_1 MountingHole_3.2mm_M3_DIN965, M3_2 MountingHole_3.2mm_M3_DIN965, Q1 BC547, Q2 BC337, Q3 BC338, Q4 BC328, U1 WeMos_mini, U2 WeMos_mini, U3 HLK-PM03, U4 TL071

Commit message: 3D and edgecut
Other:
- board size 99.2 x 98.6 mm -> 99.5 x 99.5 mm
